File: panels/alumi-blanks-v1-3U-4hp/4hp.kicad_pcb (KiCad board)
At the start: 2 copper layers, 20 x 128.5 mm, 2 parts

Commit message: feat: add new screw hole footprints and update panel KiCad files for new JLCPCB order
- Added modular-3M-screw-hole-size1-alumi-0604, modular-3M-screw-hole-size1-fit-alumi-0604, modular-3M-screw-hole-size2-alumi-0604
- Updated all panel .kicad_pcb and .kicad_pro files for 3U panels (1hp-16hp)
- Added new JLCPCB order snapshot and Gerber outputs

Co-authored-by: Copilot <223556219+Copilot@users.noreply.github.com>
Parts:
- removed ?: , 
- removed the REF** at (11.1, 3.00)
- added REF**: modular-3M-screw-hole-size2-alumi-0604, zudo-blanks:modular-3M-screw-hole-size2-alumi-0604, F.Cu at (6.04, 3.00)
- added REF**: modular-3M-screw-hole-size2-alumi-0604, zudo-blanks:modular-3M-screw-hole-size2-alumi-0604, F.Cu at (14.0, 125.5)
Changed lines of the file:
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@@
 (kicad_pcb
-	(version 20240108)
+	(version 20260206)
 	(generator "pcbnew")
-	(generator_version "8.0")
+	(generator_version "10.0")
 	(general
 		(thickness 1.6)
@@
 	(layers
 		(0 "F.Cu" signal)
-		(31 "B.Cu" signal)
-		(32 "B.Adhes" user "B.Adhesive")
-		(33 "F.Adhes" user "F.Adhesive")
-		(34 "B.Paste" user)
-		(35 "F.Paste" user)
-		(36 "B.SilkS" user "B.Silkscreen")
-		(37 "F.SilkS" user "F.Silkscreen")
-		(38 "B.Mask" user)
-		(39 "F.Mask" user)
-		(40 "Dwgs.User" user "User.Drawings")
-		(41 "Cmts.User" user "User.Comments")
-		(42 "Eco1.User" user "User.Eco1")
-		(43 "Eco2.User" user "User.Eco2")
-		(44 "Edge.Cuts" user)
-		(45 "Margin" user)
-		(46 "B.CrtYd" user "B.Courtyard")
-		(47 "F.CrtYd" user "F.Courtyard")
-		(48 "B.Fab" user)
-		(49 "F.Fab" user)
-		(50 "User.1" user)
-		(51 "User.2" user)
-		(52 "User.3" user)
-		(53 "User.4" user)
-		(54 "User.5" user)
-		(55 "User.6" user)
-		(56 "User.7" user)
-		(57 "User.8" user)
-		(58 "User.9" user)
+		(2 "B.Cu" signal)
+		(9 "F.Adhes" user "F.Adhesive")
+		(11 "B.Adhes" user "B.Adhesive")
+		(13 "F.Paste" user)
+		(15 "B.Paste" user)
+		(5 "F.SilkS" user "F.Silkscreen")
+		(7 "B.SilkS" user "B.Silkscreen")
+		(1 "F.Mask" user)
+		(3 "B.Mask" user)
+		(17 "Dwgs.User" user "User.Drawings")
+		(19 "Cmts.User" user "User.Comments")
+		(21 "Eco1.User" user "User.Eco1")
+		(23 "Eco2.User" user "User.Eco2")
+		(25 "Edge.Cuts" user)
+		(27 "Margin" user)
+		(31 "F.CrtYd" user "F.Courtyard")
+		(29 "B.CrtYd" user "B.Courtyard")
+		(35 "F.Fab" user)
+		(33 "B.Fab" user)
+		(39 "User.1" user)
+		(41 "User.2" user)
+		(43 "User.3" user)
+		(45 "User.4" user)
+		(47 "User.5" user)
+		(49 "User.6" user)
+		(51 "User.7" user)
+		(53 "User.8" user)
+		(55 "User.9" user)
 	)
 	(setup
 		(pad_to_mask_clearance 0)
 		(allow_soldermask_bridges_in_footprints no)
+		(tenting
+			(front yes)
+			(back yes)
+		)
+		(covering
+			(front no)
+			(back no)
+		)
+		(plugging
+			(front no)
+			(back no)
+		)
+		(capping no)
+		(filling no)
 		(pcbplotparams
-			(layerselection 0x00010fc_ffffffff)
-			(plot_on_all_layers_selection 0x0000000_00000000)
+			(layerselection 0x00000000_00000000_55555555_5755555a)
+			(plot_on_all_layers_selection 0x00000000_00000000_00000000_00000000)
 			(disableapertmacros no)
 			(usegerberextensions no)
@@
 			(usegerberadvancedattributes yes)
 			(creategerberjobfile yes)
-			(dashed_line_dash_ratio 12.000000)
-			(dashed_line_gap_ratio 3.000000)
+			(dashed_line_dash_ratio 12)
+			(dashed_line_gap_ratio 3)
 			(svgprecision 4)
 			(plotframeref no)
-			(viasonmask no)
 			(mode 1)
 			(useauxorigin no)
-			(hpglpennumber 1)
-			(hpglpenspeed 20)
-			(hpglpendiameter 15.000000)
 			(pdf_front_fp_property_popups yes)
 			(pdf_back_fp_property_popups yes)
+			(pdf_metadata yes)
+			(pdf_single_document no)
 			(dxfpolygonmode yes)
 			(dxfimperialunits yes)
@@
 			(psnegative no)
 			(psa4output no)
-			(plotreference yes)
-			(plotvalue yes)
-			(plotfptext yes)
-			(plotinvisibletext no)
+			(plot_black_and_white yes)
 			(sketchpadsonfab no)
+			(plotpadnumbers no)
+			(hidednponfab no)
+			(sketchdnponfab yes)
+			(crossoutdnponfab yes)
 			(subtractmaskfromsilk no)
 			(outputformat 1)
@@
 		)
 	)
-	(net 0 "")
-	(footprint "Takazudo:BlankPanelHole-M3-Alumi"
+	(footprint "zudo-blanks:modular-3M-screw-hole-size2-alumi-0604"
 		(layer "F.Cu")
-		(at 11.05 3)
+		(at 6.045 3)
 		(property "Reference" "REF**"
 			(at 0 -0.5 0)
@@
 			)
 		)
-		(property "Value" "BlankPanelHole-M3-Alumi"
+		(property "Value" "modular-3M-screw-hole-size2-alumi-0604"
 			(at 0 1 0)
 			(unlocked yes)
@@
 			)
 		)
-		(property "Footprint" "Takazudo:BlankPanelHole-M3-Alumi"
-			(at 0 0 0)
-			(unlocked yes)
-			(layer "F.Fab")
-			(hide yes)
-			(effects
-				(font
-					(size 1 1)
-					(thickness 0.15)
-				)
-			)
-		)
 		(property "Datasheet" ""
 			(at 0 0 0)
@@
 			)
 		)
-		(attr through_hole)
+		(attr smd)
+		(duplicate_pad_numbers_are_jumpers no)
 		(pad "" np_thru_hole roundrect
 			(at 0 0 90)
-			(size 3.6 10.7)
-			(drill oval 3.2 10.3)
-			(layers "F.Cu" "F.Mask")
-			(roundrect_rratio 0.5)
-		)
-	)
-	(footprint ""
+			(size 4 11.08)
+			(drill oval 3.2 10.28)
+			(layers "*.Mask")
+			(roundrect_rratio 0.4998750312)
+		)
+		(embedded_fonts no)
+	)
+	(footprint "zudo-blanks:modular-3M-screw-hole-size2-alumi-0604"
 		(layer "F.Cu")
-		(at 8.8 125.5)
-		(property "Reference" ""
-			(at 0 0 0)
+		(at 13.955 125.5)
+		(property "Reference" "REF**"
+			(at 0 -0.5 0)
+			(unlocked yes)
 			(layer "F.SilkS")
-			(effects
-				(font
-					(size 1.27 1.27)
-					(thickness 0.15)
-				)
-			)
-		)
-		(property "Value" ""
-			(at 0 0 0)
-			(layer "F.Fab")
-			(effects
-				(font
-					(size 1.27 1.27)
-					(thickness 0.15)
-				)
-			)
-		)
-		(property "Footprint" ""
-			(at 0 0 0)
-			(layer "F.Fab")
-			(hide yes)
-			(effects
-				(font
-					(size 1.27 1.27)
+			(hide yes)
+			(effects
+				(font
+					(size 1 1)
+					(thickness 0.1)
+				)
+			)
+		)
+		(property "Value" "modular-3M-screw-hole-size2-alumi-0604"
+			(at 0 1 0)
+			(unlocked yes)
+			(layer "F.Fab")
+			(hide yes)
+			(effects
+				(font
+					(size 1 1)
 					(thickness 0.15)
 				)
@@
 		(property "Datasheet" ""
 			(at 0 0 0)
-			(layer "F.Fab")
-			(hide yes)
-			(effects
-				(font
-					(size 1.27 1.27)
+			(unlocked yes)
+			(layer "F.Fab")
+			(hide yes)
+			(effects
+				(font
+					(size 1 1)
 					(thickness 0.15)
 				)
@@
 		(property "Description" ""
 			(at 0 0 0)
-			(layer "F.Fab")
-			(hide yes)
-			(effects
-				(font
-					(size 1.27 1.27)
-					(thickness 0.15)
-				)
-			)
-		)
+			(unlocked yes)
+			(layer "F.Fab")
+			(hide yes)
+			(effects
+				(font
+					(size 1 1)
+					(thickness 0.15)
+				)
+			)
+		)
+		(attr smd)
+		(duplicate_pad_numbers_are_jumpers no)
 		(pad "" np_thru_hole roundrect
 			(at 0 0 90)
-			(size 3.6 10.7)
-			(drill oval 3.2 10.3)
-			(layers "F.Cu" "In1.Cu" "In2.Cu" "In3.Cu" "In4.Cu" "In5.Cu" "In6.Cu" "In7.Cu"
-				"In8.Cu" "In9.Cu" "In10.Cu" "In11.Cu" "In12.Cu" "In13.Cu" "In14.Cu" "In15.Cu"
-				"In16.Cu" "In17.Cu" "In18.Cu" "In19.Cu" "In20.Cu" "In21.Cu" "In22.Cu"
-				"In23.Cu" "In24.Cu" "In25.Cu" "In26.Cu" "In27.Cu" "In28.Cu" "In29.Cu"
-				"In30.Cu" "F.Mask"
-			)
-			(roundrect_rratio 0.5)
-		)
+			(size 4 11.08)
+			(drill oval 3.2 10.28)
+			(layers "*.Mask")
+			(roundrect_rratio 0.4998750312)
+		)
+		(embedded_fonts no)
 	)
 	(gr_poly
@@
 			(color 35 31 32 1)
 		)
-		(fill none)
+		(fill no)
 		(layer "Edge.Cuts")
 	)
 	(gr_poly
 		(pts
+			(xy 5.700454 30.003191) (xy 0.000001 30.003191) (xy 0.000001 0.005265) (xy 5.700454 0.005265)
+		)
+		(stroke
+			(width -0.000001)
+			(type solid)
+		)
+		(fill yes)
+		(layer "User.1")
+	)
+	(gr_poly
+		(pts
+			(xy 17.450583 1.204617) (xy 0.000001 1.204617) (xy 0.000001 0.005265) (xy 17.450583 0.005265)
+		)
+		(stroke
+			(width -0.000001)
+			(type solid)
+		)
+		(fill yes)
+		(layer "User.1")
+	)
+	(gr_poly
+		(pts
 			(xy 19.852816 128.494736) (xy 1.608545 128.494736) (xy 1.608545 127.295387) (xy 19.852816 127.295387)
 		)
@@
 			(type solid)
 		)
-		(fill solid)
-		(layer "User.1")
-	)
-	(gr_poly
-		(pts
-			(xy 17.450583 1.204617) (xy 0.000001 1.204617) (xy 0.000001 0.005265) (xy 17.450583 0.005265)
-		)
-		(stroke
-			(width -0.000001)
-			(type solid)
-		)
-		(fill solid)
-		(layer "User.1")
-	)
-	(gr_poly
-		(pts
-			(xy 5.700454 30.003191) (xy 0.000001 30.003191) (xy 0.000001 0.005265) (xy 5.700454 0.005265)
-		)
-		(stroke
-			(width -0.000001)
-			(type solid)
-		)
-		(fill solid)
+		(fill yes)
 		(layer "User.1")
 	)
@@
 			(type solid)
 		)
-		(fill solid)
-		(layer "User.1")
-	)
+		(fill yes)
+		(layer "User.1")
+	)
+	(embedded_fonts no)
 )
